Commit message: add camera and world

File: robot_pnp/urdf/ur.xacro (robot description, xacro)
@@ -25,4 +25,5 @@
   -->
   <xacro:include filename="$(find robot_pnp)/urdf/ur_macro.xacro"/>
+  <xacro:include filename="$(find robot_pnp)/urdf/camera.xacro"/>
   <!--Declare arguments -->
   <xacro:arg name="joint_limit_params" default=""/>
@@ -78,3 +79,15 @@
     <origin xyz="0 0 0" rpy="0 0 0"/>
   </joint>
+  <joint name="camera_joint" type="fixed">
+    <axis xyz="0 0 0" />
+    <origin xyz="0 0 0.2" rpy="${pi} ${-pi/2} 0"/>
+    <parent link="robotiq_arg2f_base_link"/>
+    <child link="camera_link"/>
+  </joint>
+  <joint name="camera_optical_joint" type="fixed">
+    <axis xyz="0 0 0" />
+    <origin xyz="0 0 0" rpy="${-pi/2} 0 ${-pi/2}"/>
+    <parent link="camera_link"/>
+    <child link="camera_frame_optical"/>
+  </joint>
 </robot>
