Commit message: update for capturing

File: robot_pnp/urdf/blue_cube.urdf (robot description, URDF)
Before this commit: robot blue_cube, 1 links, 0 joints
Links:
- removed link base_link
- added link base_link_blue, mass 0.1; collision box size=0.08 0.08 0.08; visual box size=0.08 0.08 0.08

File: robot_pnp/urdf/green_cube.urdf (robot description, URDF)
Before this commit: robot green_cube, 1 links, 0 joints
Links:
- removed link base_link
- added link base_link_green, mass 0.1; collision box size=0.08 0.08 0.08; visual box size=0.08 0.08 0.08

File: robot_pnp/urdf/red_cube.urdf (robot description, URDF)
Before this commit: robot red_cube, 1 links, 0 joints
Links:
- removed link base_link
- added link base_link_red, mass 0.1; collision box size=0.08 0.08 0.08; visual box size=0.08 0.08 0.08

File: robot_pnp/urdf/ur_macro.xacro (robot description, xacro)
@@ -92,4 +92,20 @@
       </plugin>
     </gazebo>
+<!-- right_inner_finger_pad
+left_inner_finger_pad -->
+    <gazebo reference="right_inner_finger_pad">
+      <mu1>1000</mu1>
+      <mu2>1000</mu2>
+      <kp>1000000.0</kp>
+      <kd>100.0</kd>
+      <material>Gazebo/RedBright</material>
+    </gazebo>
+    <gazebo reference="left_inner_finger_pad">
+      <mu1>1000</mu1>
+      <mu2>1000</mu2>
+      <kp>1000000.0</kp>
+      <kd>100.0</kd>
+      <material>Gazebo/RedBright</material>
+    </gazebo>
   </xacro:macro>
 </robot>
